File: hardware/mff2-to-4ffnano -left v1.0/mff2-to-4ffnano-left v1.0.brd (EAGLE design)
At the start: 47.8 x 13 mm, 2 parts

Commit message: Create variants file
Parts:
- moved U$1 4.83 mm to (26.5, 14.3), turned to 180 degrees
Routing:
- net GND: track 113.3 -> 127.9 mm, vias 36 -> 32
- net SIM_DATA: track 34.4 -> 40.8 mm, vias 0 -> 2
- net SIM_CLK: track 48.4 -> 52.9 mm, vias 2 -> 0
- net SIM_RST: track 47.3 -> 51.5 mm
- net SIM_VCC: track 85.8 -> 85.4 mm, vias 0 -> 2
Other:
- board size 47.8 x 13 mm -> 48.1 x 13.8 mm
- board text added: "MFF2 to 4FF Nano-left V1.0"
- board text removed: "MFF2 to 4FF Nano V1.0"
