File: hardware/mff2-to-4ffnano-top v1.0/mff2-to-4ffnano-top v1.0.brd (EAGLE design)
At the start: 47.8 x 13 mm, 2 parts

Commit message: Create variants file
Parts:
- turned U$1 to 270 degrees
Routing:
- net GND: track 113.3 -> 41.8 mm, vias 36 -> 33
- net SIM_VCC: track 85.8 -> 92.0 mm, vias 0 -> 2
- net SIM_DATA: track 34.4 -> 37.8 mm, vias 0 -> 2
- net SIM_CLK: track 48.4 -> 48.6 mm, vias 2 -> 0
Other:
- board text added: "36层，加补强板"
- board text added: "MFF2 to 4FF Nano-top V1.0"
- board text removed: "MFF2 to 4FF Nano V1.0"
